File: PCB/nRF52-BLEUart-module/board.sch (EAGLE design)
At the start: 43 parts, among them J1 USB-A_PTH_MALE, U1 CH340E, U2 NRF52832, Y1 32MHz_2016, Y2 32.768kHz

Commit message: final PCB for V1.0
Parts:
- C15, C16: value (none) -> DNP
- D3: LCSC C2286 -> C72038
- D4, D5, D6: LCSC C72038 -> C2286
- JP1: device angrypig7-Connectors-PinHeads:PINHD-1X4/90 -> angrypig7-Connectors-PinHeads:PINHD-1X4NOSILK
- JP2: value 3V3 5V -> 5V 3V3
- R1: value 10k -> 15k; LCSC C25744 -> C25756
- U2: JLC_ROTATION 180 -> 270
Changed lines of the file:
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@@
 <part name="GND3" library="angrypig7-Symbols" deviceset="GND" device=""/>
 <part name="U2" library="angrypig7-IC-MCU" deviceset="NRF52832" device="" package3d_urn="urn:adsk.eagle:package:25776865/5">
-<attribute name="JLC_ROTATION" value="180"/>
+<attribute name="JLC_ROTATION" value="270"/>
 <attribute name="LCSC" value="C77540"/>
 </part>
@@
 </part>
 <part name="GND19" library="angrypig7-Symbols" deviceset="GND" device=""/>
-<part name="C15" library="angrypig7-RCL" deviceset="C-NON-POL" device="C0402" package3d_urn="urn:adsk.eagle:package:23626/2">
+<part name="C15" library="angrypig7-RCL" deviceset="C-NON-POL" device="C0402" package3d_urn="urn:adsk.eagle:package:23626/2" value="DNP">
 <spice>
 <pinmapping spiceprefix="C">
@@
 <attribute name="LCSC" value="C17168"/>
 </part>
-<part name="C16" library="angrypig7-RCL" deviceset="C-NON-POL" device="C0402" package3d_urn="urn:adsk.eagle:package:23626/2">
+<part name="C16" library="angrypig7-RCL" deviceset="C-NON-POL" device="C0402" package3d_urn="urn:adsk.eagle:package:23626/2" value="DNP">
 <spice>
 <pinmapping spiceprefix="C">
@@
 <part name="SUPPLY15" library="angrypig7-Symbols" deviceset="3V3" device=""/>
 <part name="GND25" library="angrypig7-Symbols" deviceset="GND" device=""/>
-<part name="R1" library="angrypig7-RCL" deviceset="R" device="R0402" package3d_urn="urn:adsk.eagle:package:23547/3" value="10k">
-<spice>
-<pinmapping spiceprefix="R">
-<pinmap gate="G$1" pin="1" pinorder="1"/>
-<pinmap gate="G$1" pin="2" pinorder="2"/>
-</pinmapping>
-</spice>
-<attribute name="LCSC" value="C25744"/>
+<part name="R1" library="angrypig7-RCL" deviceset="R" device="R0402" package3d_urn="urn:adsk.eagle:package:23547/3" value="15k">
+<spice>
+<pinmapping spiceprefix="R">
+<pinmap gate="G$1" pin="1" pinorder="1"/>
+<pinmap gate="G$1" pin="2" pinorder="2"/>
+</pinmapping>
+</spice>
+<attribute name="LCSC" value="C25756"/>
 </part>
 <part name="D3" library="angrypig7-Diodes" deviceset="LED" device="_0603" package3d_urn="urn:adsk.eagle:package:22866870/2" value="PWR">
-<attribute name="LCSC" value="C2286"/>
+<attribute name="LCSC" value="C72038"/>
 </part>
 <part name="GND26" library="angrypig7-Symbols" deviceset="GND" device=""/>
@@
 </part>
 <part name="D4" library="angrypig7-Diodes" deviceset="LED" device="_0603" package3d_urn="urn:adsk.eagle:package:22866870/2" value="0603">
-<attribute name="LCSC" value="C72038"/>
+<attribute name="LCSC" value="C2286"/>
 </part>
 <part name="R4" library="angrypig7-RCL" deviceset="R" device="R0402" package3d_urn="urn:adsk.eagle:package:23547/3" value="10k">
@@
 </part>
 <part name="D5" library="angrypig7-Diodes" deviceset="LED" device="_0603" package3d_urn="urn:adsk.eagle:package:22866870/2" value="0603">
-<attribute name="LCSC" value="C72038"/>
+<attribute name="LCSC" value="C2286"/>
 </part>
 <part name="FRAME2" library="angrypig7-Frames" deviceset="FRAME-A3L" device=""/>
 <part name="FRAME1" library="angrypig7-Frames" deviceset="FRAME-A3L" device=""/>
-<part name="JP1" library="angrypig7-Connectors-PinHeads" deviceset="PINHD-1X4" device="/90" package3d_urn="urn:adsk.eagle:package:22404/2" value="V  G Tx Rx"/>
-<part name="JP2" library="angrypig7-Jumpers" deviceset="JUMPER-SMT_3_1-NC_TRACE" device="_NO-SILK" package3d_urn="urn:adsk.eagle:package:39287/1" value="3V3 5V "/>
+<part name="JP1" library="angrypig7-Connectors-PinHeads" deviceset="PINHD-1X4" device="NOSILK" value="V  G Tx Rx"/>
+<part name="JP2" library="angrypig7-Jumpers" deviceset="JUMPER-SMT_3_1-NC_TRACE" device="_NO-SILK" package3d_urn="urn:adsk.eagle:package:39287/1" value=" 5V 3V3"/>
 <part name="SUPPLY20" library="angrypig7-Symbols" deviceset="5V" device=""/>
 <part name="GND7" library="angrypig7-Symbols" deviceset="GND" device=""/>
@@
 </part>
 <part name="D6" library="angrypig7-Diodes" deviceset="LED" device="_0603" package3d_urn="urn:adsk.eagle:package:22866870/2" value="0603">
-<attribute name="LCSC" value="C72038"/>
+<attribute name="LCSC" value="C2286"/>
 </part>
 <part name="GND32" library="angrypig7-Symbols" deviceset="GND" device=""/>
