File: PCB/nRF52-BLEUart-module/board.sch (EAGLE design)
At the start: 43 parts, among them J1 USB-A_PTH_MALE, U1 CH340E, U2 NRF52832, Y1 32MHz_2016, Y2 32.768kHz

Commit message: V1.1.0 update
Parts:
- JP1: value V G Tx Rx -> Rx Tx G V
- R1: value 15k -> 7.5k; LCSC C25756 -> C25918
- U$1: device angrypig7-Antennas:INVERTED_F_2.4GHZ_TI-AN043_L -> angrypig7-Antennas:INVERTED_F_2.4GHZ_TI-AN043_L_SHORT
Changed lines of the file:
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@@
 <attribute name="CDESIGNER" value="Kihun Song"/>
 <attribute name="CNAME" value="nRF52-BLEUart-module"/>
-<attribute name="CREVISION" value="V1.0.0"/>
+<attribute name="CREVISION" value="V1.1.0"/>
 </attributes>
 <variantdefs>
@@
 <part name="SUPPLY15" library="angrypig7-Symbols" deviceset="3V3" device=""/>
 <part name="GND25" library="angrypig7-Symbols" deviceset="GND" device=""/>
-<part name="R1" library="angrypig7-RCL" deviceset="R" device="R0402" package3d_urn="urn:adsk.eagle:package:23547/3" value="15k">
+<part name="R1" library="angrypig7-RCL" deviceset="R" device="R0402" package3d_urn="urn:adsk.eagle:package:23547/3" value="7.5k">
 <spice>
 <pinmapping spiceprefix="R">
@@
 </pinmapping>
 </spice>
-<attribute name="LCSC" value="C25756"/>
+<attribute name="LCSC" value="C25918"/>
 </part>
 <part name="D3" library="angrypig7-Diodes" deviceset="LED" device="_0603" package3d_urn="urn:adsk.eagle:package:22866870/2" value="PWR">
@@
 <part name="FRAME2" library="angrypig7-Frames" deviceset="FRAME-A3L" device=""/>
 <part name="FRAME1" library="angrypig7-Frames" deviceset="FRAME-A3L" device=""/>
-<part name="JP1" library="angrypig7-Connectors-PinHeads" deviceset="PINHD-1X4" device="NOSILK" value="V  G Tx Rx"/>
+<part name="JP1" library="angrypig7-Connectors-PinHeads" deviceset="PINHD-1X4" device="NOSILK" value="Rx Tx G  V"/>
 <part name="JP2" library="angrypig7-Jumpers" deviceset="JUMPER-SMT_3_1-NC_TRACE" device="_NO-SILK" package3d_urn="urn:adsk.eagle:package:39287/1" value=" 5V 3V3"/>
 <part name="SUPPLY20" library="angrypig7-Symbols" deviceset="5V" device=""/>
@@
 <part name="GND29" library="angrypig7-Symbols" deviceset="GND" device=""/>
 <part name="JP4" library="angrypig7-Connectors-PinHeads" deviceset="PINHD-1X5" device="-NOSILK"/>
-<part name="U$1" library="angrypig7-Antennas" deviceset="INVERTED_F_2.4GHZ_TI-AN043" device="_L" value="ANT"/>
+<part name="U$1" library="angrypig7-Antennas" deviceset="INVERTED_F_2.4GHZ_TI-AN043" device="_L_SHORT" value="ANT"/>
 <part name="GND30" library="angrypig7-Symbols" deviceset="GND" device=""/>
 <part name="SUPPLY14" library="angrypig7-Symbols" deviceset="VCCIO" device=""/>
